File: f0-study-board/f0-study-board/f0-study-board.sch (KiCad schematic (older format))
At the start: 26 parts, among them J1 PinHeader-18pin, J2 PinHeader-18pin, J3 USB_B_Micro, J4 SWD, SW1 SW_Reset, U1 STM32F091CBT6, U2 XC6206P332MR, Y1 8MHz

Commit message: Had to choose another mcu
Parts:
- removed C5: 100n, Capacitor_SMD:C_0402_1005Metric, symbol Device:C_Small
- removed U1: STM32F091CBT6, Package_QFP:LQFP-48_7x7mm_P0.5mm, symbol MCU_ST_STM32F0:STM32F091CBTx
- added U1: STM32F030C8T6, Package_QFP:LQFP-48_7x7mm_P0.5mm, symbol MCU_ST_STM32F0:STM32F030C8Tx
Connections:
- net +3.3VA: now also U1.9 (VDDA)
- net +3V3: now also U1.1 (VDD), U1.24 (VDD), U1.48 (VDD)
- net BOOT0: now also U1.44 (BOOT0)
- net GND: now also U1.23 (VSS), U1.47 (VSS), U1.8 (VSSA)
- net NRST: now also U1.7 (NRST)
- net OSC_IN: now also U1.5 (PF0)
- net OSC_OUT: now also U1.6 (PF1)
- net PA0: now also U1.10 (PA0)
- net PA1: now also U1.11 (PA1)
- net PA10: now also U1.31 (PA10)
- net PA11: now also U1.32 (PA11)
- net PA12: now also U1.33 (PA12)
- net PA15: now also U1.38 (PA15)
- net PA2: now also U1.12 (PA2)
- net PA3: now also U1.13 (PA3)
- net PA4: now also U1.14 (PA4)
- net PA5: now also U1.15 (PA5)
- net PA6: now also U1.16 (PA6)
- net PA7: now also U1.17 (PA7)
- net PA8: now also U1.29 (PA8)
- net PA9: now also U1.30 (PA9)
- net PB0: now also U1.18 (PB0)
- net PB1: now also U1.19 (PB1)
- net PB10: now also U1.21 (PB10)
- net PB11: now also U1.22 (PB11)
- net PB12: now also U1.25 (PB12)
- net PB13: now also U1.26 (PB13)
- net PB14: now also U1.27 (PB14)
- net PB15: now also U1.28 (PB15)
- net PB2: now also U1.20 (PB2)
- net PB3: now also U1.39 (PB3)
- net PB4: now also U1.40 (PB4)
- net PB5: now also U1.41 (PB5)
- net PB6: now also U1.42 (PB6)
- net PB7: now also U1.43 (PB7)
- net PB8: now also U1.45 (PB8)
- net PB9: now also U1.46 (PB9)
- net SWCLK: now also U1.37 (PA14)
- net SWDIO: now also U1.34 (PA13)
- no-connect marks 10 -> 13
Other:
- moved on the sheet: C10, C8, C9, R1, SW1, Y1

Commit message: Board gerbers sent
Parts:
- C1: LCSC (none) -> C1779; LCSC Part # C1779 -> (none)
- C10, C9: LCSC (none) -> C1570; LCSC Part # C1570 -> (none)
- C11, C12: LCSC (none) -> C28323; LCSC Part # C28323 -> (none)
- C2, C3, C4, C7, C8: LCSC (none) -> C307331; LCSC Part # C307331 -> (none)
- C6: LCSC (none) -> C52923; LCSC Part # C52923 -> (none)
- D2: LCSC (none) -> C72041; LCSC Part # C72041 -> (none)
- FB1: LCSC (none) -> C74325; LCSC Part # C74325 -> (none)
- J3: LCSC (none) -> C132560; LCSC Part # C132560 -> (none)
- L1: LCSC (none) -> C18830; LCSC Part # C18830 -> (none)
- R1: LCSC (none) -> C25744; LCSC Part # C25744 -> (none)
- R2: LCSC (none) -> C11702; LCSC Part # C11702 -> (none)
- SW1: LCSC (none) -> C115357; LCSC Part # C115357 -> (none)
- U1: LCSC (none) -> C23922; LCSC Part # C23922 -> (none)
- U2: LCSC (none) -> C5446; LCSC Part # C5446 -> (none)
- Y1: LCSC (none) -> C115962; LCSC Part # C115962 -> (none)
Changed lines of the file:
@@
 F 2 "Capacitor_SMD:C_0805_2012Metric" H 1100 1250 50  0001 C CNN
 F 3 "~" H 1100 1250 50  0001 C CNN
-F 4 "C1779" H 1100 1250 50  0001 C CNN "LCSC Part #"
+F 4 "C1779" H 1100 1250 50  0001 C CNN "LCSC"
 	1    1100 1250
 	1    0    0    -1
@@
 F 2 "Capacitor_SMD:C_0402_1005Metric" H 1500 1250 50  0001 C CNN
 F 3 "~" H 1500 1250 50  0001 C CNN
-F 4 "C307331" H 1500 1250 50  0001 C CNN "LCSC Part #"
+F 4 "C307331" H 1500 1250 50  0001 C CNN "LCSC"
 	1    1500 1250
 	1    0    0    -1
@@
 F 2 "Capacitor_SMD:C_0402_1005Metric" H 1900 1250 50  0001 C CNN
 F 3 "~" H 1900 1250 50  0001 C CNN
-F 4 "C307331" H 1900 1250 50  0001 C CNN "LCSC Part #"
+F 4 "C307331" H 1900 1250 50  0001 C CNN "LCSC"
 	1    1900 1250
 	1    0    0    -1
@@
 F 2 "Capacitor_SMD:C_0402_1005Metric" H 2300 1250 50  0001 C CNN
 F 3 "~" H 2300 1250 50  0001 C CNN
-F 4 "C307331" H 2300 1250 50  0001 C CNN "LCSC Part #"
+F 4 "C307331" H 2300 1250 50  0001 C CNN "LCSC"
 	1    2300 1250
 	1    0    0    -1
@@
 F 2 "Inductor_SMD:L_0402_1005Metric" H 3700 1100 50  0001 C CNN
 F 3 "~" H 3700 1100 50  0001 C CNN
-F 4 "C18830" H 3700 1100 50  0001 C CNN "LCSC Part #"
+F 4 "C18830" H 3700 1100 50  0001 C CNN "LCSC"
 	1    3700 1100
 	0    -1   -1   0
@@
 F 2 "Capacitor_SMD:C_0402_1005Metric" H 4400 1250 50  0001 C CNN
 F 3 "~" H 4400 1250 50  0001 C CNN
-F 4 "C307331" H 4400 1250 50  0001 C CNN "LCSC Part #"
+F 4 "C307331" H 4400 1250 50  0001 C CNN "LCSC"
 	1    4400 1250
 	1    0    0    -1
@@
 F 2 "Capacitor_SMD:C_0402_1005Metric" H 4000 1250 50  0001 C CNN
 F 3 "~" H 4000 1250 50  0001 C CNN
-F 4 "C52923" H 4000 1250 50  0001 C CNN "LCSC Part #"
+F 4 "C52923" H 4000 1250 50  0001 C CNN "LCSC"
 	1    4000 1250
 	1    0    0    -1
@@
 F 2 "Button_Switch_SMD:SW_Push_SPST_NO_Alps_SKRK" H 2150 3500 50  0001 C CNN
 F 3 "~" H 2150 3500 50  0001 C CNN
-F 4 "C115357" H 2150 3300 50  0001 C CNN "LCSC Part #"
+F 4 "C115357" H 2150 3300 50  0001 C CNN "LCSC"
 	1    2150 3300
 	1    0    0    -1
@@
 F 2 "Resistor_SMD:R_0402_1005Metric" H 1600 4700 50  0001 C CNN
 F 3 "~" H 1600 4700 50  0001 C CNN
-F 4 "C25744" H 1600 4700 50  0001 C CNN "LCSC Part #"
+F 4 "C25744" H 1600 4700 50  0001 C CNN "LCSC"
 	1    1600 4700
 	1    0    0    -1
@@
 F 2 "Capacitor_SMD:C_0402_1005Metric" H 2450 3450 50  0001 C CNN
 F 3 "~" H 2450 3450 50  0001 C CNN
-F 4 "C307331" H 2450 3450 50  0001 C CNN "LCSC Part #"
+F 4 "C307331" H 2450 3450 50  0001 C CNN "LCSC"
 	1    2450 3450
 	1    0    0    -1
@@
 F 2 "Crystal:Crystal_SMD_5032-2Pin_5.0x3.2mm" H 2250 5150 50  0001 C CNN
 F 3 "~" H 2250 5150 50  0001 C CNN
-F 4 "C115962" H 2250 5150 50  0001 C CNN "LCSC Part #"
+F 4 "C115962" H 2250 5150 50  0001 C CNN "LCSC"
 	1    2250 5150
 	1    0    0    -1
@@
 F 2 "Capacitor_SMD:C_0402_1005Metric" H 2000 5400 50  0001 C CNN
 F 3 "~" H 2000 5400 50  0001 C CNN
-F 4 "C1570" H 2000 5400 50  0001 C CNN "LCSC Part #"
+F 4 "C1570" H 2000 5400 50  0001 C CNN "LCSC"
 	1    2000 5400
 	1    0    0    -1
@@
 F 2 "Capacitor_SMD:C_0402_1005Metric" H 2500 5400 50  0001 C CNN
 F 3 "~" H 2500 5400 50  0001 C CNN
-F 4 "C1570" H 2500 5400 50  0001 C CNN "LCSC Part #"
+F 4 "C1570" H 2500 5400 50  0001 C CNN "LCSC"
 	1    2500 5400
 	1    0    0    -1
@@
 F 2 "LED_SMD:LED_0603_1608Metric" V 5750 6150 50  0001 C CNN
 F 3 "~" V 5750 6150 50  0001 C CNN
-F 4 "C72041" H 5750 6150 50  0001 C CNN "LCSC Part #"
+F 4 "C72041" H 5750 6150 50  0001 C CNN "LCSC"
 	1    5750 6150
 	-1   0    0    1
@@
 F 2 "Resistor_SMD:R_0402_1005Metric" H 6050 6400 50  0001 C CNN
 F 3 "~" H 6050 6400 50  0001 C CNN
-F 4 "C11702" H 6050 6400 50  0001 C CNN "LCSC Part #"
+F 4 "C11702" H 6050 6400 50  0001 C CNN "LCSC"
 	1    6050 6400
 	1    0    0    -1
@@
 F 2 "Connector_USB:USB_Micro-B_Molex_47346-0001" H 8550 1500 50  0001 C CNN
 F 3 "~" H 8550 1500 50  0001 C CNN
-F 4 "C132560" H 8400 1550 50  0001 C CNN "LCSC Part #"
+F 4 "C132560" H 8400 1550 50  0001 C CNN "LCSC"
 	1    8400 1550
 	1    0    0    -1
@@
 F 2 "Inductor_SMD:L_0603_1608Metric" V 9030 1350 50  0001 C CNN
 F 3 "~" H 9100 1350 50  0001 C CNN
-F 4 "C74325" H 9100 1350 50  0001 C CNN "LCSC Part #"
+F 4 "C74325" H 9100 1350 50  0001 C CNN "LCSC"
 	1    9100 1350
 	0    1    1    0
@@
 F 2 "Capacitor_SMD:C_0805_2012Metric" H 9250 1700 50  0001 C CNN
 F 3 "~" H 9250 1700 50  0001 C CNN
-F 4 "C28323" H 9250 1700 50  0001 C CNN "LCSC Part #"
+F 4 "C28323" H 9250 1700 50  0001 C CNN "LCSC"
 	1    9250 1700
 	1    0    0    -1
@@
 F 2 "Package_TO_SOT_SMD:SOT-23" H 9900 1575 50  0001 C CIN
 F 3 "https://www.torexsemi.com/file/xc6206/XC6206.pdf" H 9900 1350 50  0001 C CNN
-F 4 "C5446" H 9900 1350 50  0001 C CNN "LCSC Part #"
+F 4 "C5446" H 9900 1350 50  0001 C CNN "LCSC"
 	1    9900 1350
 	1    0    0    -1
@@
 F 2 "Capacitor_SMD:C_0805_2012Metric" H 10550 1700 50  0001 C CNN
 F 3 "~" H 10550 1700 50  0001 C CNN
-F 4 "C28323" H 10550 1700 50  0001 C CNN "LCSC Part #"
+F 4 "C28323" H 10550 1700 50  0001 C CNN "LCSC"
 	1    10550 1700
 	1    0    0    -1
@@
 F 2 "Package_QFP:LQFP-48_7x7mm_P0.5mm" H 3550 3650 50  0001 R CNN
 F 3 "http://www.st.com/st-web-ui/static/active/en/resource/technical/document/datasheet/DM00088500.pdf" H 4050 5150 50  0001 C CNN
-F 4 "C23922" H 4050 5150 50  0001 C CNN "LCSC Part #"
+F 4 "C23922" H 4050 5150 50  0001 C CNN "LCSC"
 	1    4050 5150
 	1    0    0    -1
